File: promicro_rp2040_pcbholder_wiredver/promicro_rp2040_pcbholder_wiredver.kicad_sch (KiCad schematic)
At the start: 8 parts, among them J1 Conn_01x08_Pin, J2 Conn_01x08_Pin, J3 Conn_01x08_Pin, J4 Conn_01x08_Pin, U1 RP2040_Pro_Micro, U2 TRRS, U3 RP2040_Pro_Micro, U4 TRRS

Commit message: schematic naming
Connections:
- net Col1 is gone; now on net RCol1: J1.1 (Pin_1), U1.6 (GP2)
- net Col2 is gone; now on net RCol2: J1.2 (Pin_2), U1.7 (GP3)
- net Col3 is gone; now on net RCol3: J1.3 (Pin_3), U1.8 (GP4)
- net Col4 is gone; now on net RCol4: J1.4 (Pin_4), U1.9 (GP5)
- net Col5 is gone; now on net RCol5: J1.5 (Pin_5), U1.10 (GP6)
- net Col6 is gone; now on net RCol6: J1.6 (Pin_6), U1.11 (GP7)
- net Col7 is gone; now on net RCol7: J1.7 (Pin_7), U1.12 (GP8)
- net Col8 is gone; now on net RCol8: J1.8 (Pin_8), U1.13 (GP9)
- net Row1 is gone; now on net RRow1: J2.1 (Pin_1), U1.26 (GP29)
- net Row2 is gone; now on net RRow2: J2.2 (Pin_2), U1.25 (GP28)
- net Row3 is gone; now on net RRow3: J2.3 (Pin_3), U1.24 (GP27)
- net Row4 is gone; now on net RRow4: J2.4 (Pin_4), U1.23 (GP26)
- net Row5 is gone; now on net RRow5: J2.5 (Pin_5), U1.22 (GP22)
- net Row6 is gone; now on net RRow6: J2.6 (Pin_6), U1.21 (GP20)
- net Row7 is gone; now on net RRow7: J2.7 (Pin_7), U1.20 (GP23)
- net Row8 is gone; now on net RRow8: J2.8 (Pin_8), U1.19 (GP21)
- net LData: now also U3.2 (GP0), U4.4 (RING2); no longer U1.2 (GP0), U2.4 (RING2)
- net LGND: now also U3.29 (GND), U4.1 (SLEEVE); no longer U1.5 (GND), U2.1 (SLEEVE)
- net LVCC: now also U3.27 (3.3v), U4.2 (TIP); no longer U1.27 (3.3v), U2.2 (TIP)
- net RCol1: no longer J3.1 (Pin_1), U3.6 (GP2)
- net RCol2: no longer J3.2 (Pin_2), U3.7 (GP3)
- net RCol3: no longer J3.3 (Pin_3), U3.8 (GP4)
- net RCol4: no longer J3.4 (Pin_4), U3.9 (GP5)
- net RCol5: no longer J3.5 (Pin_5), U3.10 (GP6)
- net RCol6: no longer J3.6 (Pin_6), U3.11 (GP7)
- net RCol7: no longer J3.7 (Pin_7), U3.12 (GP8)
- net RCol8: no longer J3.8 (Pin_8), U3.13 (GP9)
- net RData: now also U1.2 (GP0), U2.4 (RING2); no longer U3.2 (GP0), U4.4 (RING2)
- net RGND: now also U1.5 (GND), U2.1 (SLEEVE); no longer U3.29 (GND), U4.1 (SLEEVE)
- net RRow1: no longer J4.1 (Pin_1), U3.26 (GP29)
- net RRow2: no longer J4.2 (Pin_2), U3.25 (GP28)
- net RRow3: no longer J4.3 (Pin_3), U3.24 (GP27)
- net RRow4: no longer J4.4 (Pin_4), U3.23 (GP26)
- net RRow5: no longer J4.5 (Pin_5), U3.22 (GP22)
- net RRow6: no longer J4.6 (Pin_6), U3.21 (GP20)
- net RRow7: no longer J4.7 (Pin_7), U3.20 (GP23)
- net RRow8: no longer J4.8 (Pin_8), U3.19 (GP21)
- net RVCC: now also U1.27 (3.3v), U2.2 (TIP); no longer U3.27 (3.3v), U4.2 (TIP)
- new net LCol1: J3.1 (Pin_1), U3.6 (GP2)
- new net LCol2: J3.2 (Pin_2), U3.7 (GP3)
- new net LCol3: J3.3 (Pin_3), U3.8 (GP4)
- new net LCol4: J3.4 (Pin_4), U3.9 (GP5)
- new net LCol5: J3.5 (Pin_5), U3.10 (GP6)
- new net LCol6: J3.6 (Pin_6), U3.11 (GP7)
- new net LCol7: J3.7 (Pin_7), U3.12 (GP8)
- new net LCol8: J3.8 (Pin_8), U3.13 (GP9)
- new net LRow1: J4.1 (Pin_1), U3.26 (GP29)
- new net LRow2: J4.2 (Pin_2), U3.25 (GP28)
- new net LRow3: J4.3 (Pin_3), U3.24 (GP27)
- new net LRow4: J4.4 (Pin_4), U3.23 (GP26)
- new net LRow5: J4.5 (Pin_5), U3.22 (GP22)
- new net LRow6: J4.6 (Pin_6), U3.21 (GP20)
- new net LRow7: J4.7 (Pin_7), U3.20 (GP23)
- new net LRow8: J4.8 (Pin_8), U3.19 (GP21)
- no-connect marks 8 -> 16
Other:
- moved on the sheet: J1, J2, J3, J4, U1, U2, U3, U4

Commit message: initial design done. Ordered for testing
Parts:
- J1, J2, J3, J4: footprint Connector_PinHeader_2.54mm:PinHeader_1x08_P2.54mm_Vertical -> #footprint:PinHeader_1x08_P2.54mm_Vertical_rev2
Changed lines of the file:
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@@
 			)
 		)
-		(property "Footprint" "Connector_PinHeader_2.54mm:PinHeader_1x08_P2.54mm_Vertical"
+		(property "Footprint" "#footprint:PinHeader_1x08_P2.54mm_Vertical_rev2"
 			(at 35.56 73.66 0)
 			(effects
@@
 			)
 		)
-		(property "Footprint" "Connector_PinHeader_2.54mm:PinHeader_1x08_P2.54mm_Vertical"
+		(property "Footprint" "#footprint:PinHeader_1x08_P2.54mm_Vertical_rev2"
 			(at 106.68 73.66 0)
 			(effects
@@
 			)
 		)
-		(property "Footprint" "Connector_PinHeader_2.54mm:PinHeader_1x08_P2.54mm_Vertical"
+		(property "Footprint" "#footprint:PinHeader_1x08_P2.54mm_Vertical_rev2"
 			(at 165.1 76.2 0)
 			(effects
@@
 			)
 		)
-		(property "Footprint" "Connector_PinHeader_2.54mm:PinHeader_1x08_P2.54mm_Vertical"
+		(property "Footprint" "#footprint:PinHeader_1x08_P2.54mm_Vertical_rev2"
 			(at 236.22 76.2 0)
 			(effects
